File: nTerm2-s-sd.kicad_pcb (KiCad board)
At the start: 2 copper layers, 147.3 x 55.9 mm, 117 parts, among them J1 VGA, J2 Keyboard, J3 Mouse, J4 Speaker, J5 DE9_Plug_MountingHoles, J6 USB_C_Receptacle_USB2.0_16P, J7 Micro_SD_Card_Det1, K1 IM41 3V, K2 IM41 3V, K3 IM41 3V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

Commit message: If we move the DFLT button to the GPIO extender, we can use the input for the INT signal. And if we connected the SD DETECT output to the GPIO extender, we can detect card changes. And we still have 3 GPIO extentions left for other stuff. This seems doable... But we are further away from the default FABGL and uTerm2-S firmwares than with uTerm2-S now. So that means more documentation...
Parts:
- added R42: 12K, Resistor_SMD:R_0603_1608Metric_Pad0.98x0.95mm_HandSolder, F.Cu at (225.1, 66.0)
Connections:
- J2 pad 7: (no net) -> GND
- J3 pad 7: (no net) -> GND
- J4 pad R: (no net) -> unconnected-(J4-3-PadR)
- J4 pad RN: (no net) -> unconnected-(J4-5-PadRN)
- J7 pad 10: unconnected-(J7-SHIELD-Pad10) -> GND
- J7 pad 9: unconnected-(J7-DET-Pad9) -> SD_DETECT
- R28 pad 1: Net-(U1-IO39-_{ADC1_3/SENSVN}) -> Net-(U7-GP3)
- R29 pad 2: Net-(U1-IO39-_{ADC1_3/SENSVN}) -> Net-(U7-GP3)
- U1 pad 5: Net-(U1-IO39-_{ADC1_3/SENSVN}) -> IO_INT
- U6 pad 2: RAM_SD0 -> RAM_SD0/SPI_MISO
- U6 pad 3: RAM_SD3 -> RAM_SD3/SPI_WP
- U6 pad 5: RAM_SD1 -> RAM_SD1/SPI_MOSI
- U6 pad 6: RAM_CLK -> RAM_CLK/SPI_CLK
- U6 pad 7: RAM_SD2 -> RAM_SD2/SPI_HD
- U7 pad 12: unconnected-(U7-GP3-Pad12) -> Net-(U7-GP3)
- U7 pad 13: unconnected-(U7-GP4-Pad13) -> SD_DETECT
- U7 pad 8: unconnected-(U7-INT-Pad8) -> IO_INT
Routing:
- net Net-(U1-IO39-_{ADC1_3/SENSVN}): track 45.5 -> 0.00 mm, vias 2 -> 0
- net (no net): track 0.00 -> 45.5 mm, vias 0 -> 2
