File: nTerm2-s-sd.kicad_sch (KiCad schematic)
At the start: 117 parts, among them J1 VGA, J2 Keyboard, J3 Mouse, J4 Speaker, J5 DE9_Plug_MountingHoles, J6 USB_C_Receptacle_USB2.0_16P, J7 Micro_SD_Card_Det1, K1 IM41 3V, K2 IM41 3V, K3 IM41 3V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

Commit message: If we move the DFLT button to the GPIO extender, we can use the input for the INT signal. And if we connected the SD DETECT output to the GPIO extender, we can detect card changes. And we still have 3 GPIO extentions left for other stuff. This seems doable... But we are further away from the default FABGL and uTerm2-S firmwares than with uTerm2-S now. So that means more documentation...
Parts:
- added R42: 12K, Resistor_SMD:R_0603_1608Metric_Pad0.98x0.95mm_HandSolder, symbol Device:R
Connections:
- net RAM_CLK is gone; now on net RAM_CLK/SPI_CLK: U6.6 (SCLK)
- net RAM_SD0 is gone; now on net RAM_SD0/SPI_MISO: U6.2 (SO/SIO)
- net RAM_SD1 is gone; now on net RAM_SD1/SPI_MOSI: U6.5 (SI/SIO)
- net RAM_SD2 is gone; now on net RAM_SD2/SPI_HD: U6.7 (SIO3)
- net RAM_SD3 is gone; now on net RAM_SD3/SPI_WP: U6.3 (SIO2)
- net +3V3: now also R42.1
- net GND: now also J2.7, J3.7, J7.10 (SHIELD)
- net at R28.1, R29.2: now also U7.12 (GP3); no longer U1.5 (IO39-_{ADC1_3/SENSVN})
- net SD_DETECT: now reaches U7.13 (GP4)
- net SD_DETECT: now also J7.9 (DET), R42.2
- net IO_INT: now reaches U7.8 (INT)
- net IO_INT: now also U1.5 (IO39-_{ADC1_3/SENSVN})
- no-connect marks 35 -> 39
Other:
- moved on the sheet: C28, C31, C32, C33, R39, U6, U7
